File: scheme/afc-smm/analog.brd (EAGLE design)
At the start: 80 x 80 mm, 89 parts, among them IC1 OP1177R, IC10 LM2931-5.0, IC11 OP184, IC12 DAC8551, IC13 REF3033, IC14 317EMP, IC15 317EMP, IC2 TL082D, IC3 AD8515RJ, IC4 AD8615RJ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

Commit message: it is work! go to add pid_controller
Connections:
- net N$34 renamed 30V
