File: scheme/afc-smm/analog.sch (EAGLE design)
At the start: 85 parts, among them IC1 OP1177R, IC10 LM2931-5.0, IC11 OP184, IC12 DAC8551, IC13 REF3033, IC14 317EMP, IC15 317EMP, IC2 TL082D, IC3 AD8515RJ, IC4 AD8615RJ, IC5 AD8221R, IC6 AD7476, IC7 REF3033, IC8 LM337LM, IC9 317EMP, J1 22-27-2031-03, J2 22-27-2021-02, Q1 IRLML2803, X1 1-227161-0, X2 1-227161-0

Commit message: make analog out schematics, draw most of brd
Parts:
- added D4, D5: 1N4148WS, afc-smm:1N4148WS
- C14: device rcl:C-EUC0603 -> rcl:CPOL-EUSMCA
- SV1: device con-lstb:MA08-2W -> con-lstb:MA10-2W
- X1, X2: device con-coax:1-227161-0 -> afc-smm:1-227161-0
Connections:
- new net N$14: IC6.SCLK, SV1.1
- new net N$21: IC6.SDATA, SV1.3
- new net N$22: IC6.!CS, SV1.5
- new net N$23: B2.AC1, J2-2.S
- new net N$26: R27.1, SV1.2
- new net N$31: B2.+, C13.+, D4.C, IC14.VI
- new net N$32: C11.+, C12.1, D5.A, IC13.IN, IC15.VO, R20.2, TP9.PP
- new net N$33: IC14.ADJ, R6.1, R7.2
- new net N$34: C10.1, C9.+, D4.A, D5.C, IC11.+VS, IC14.VO, IC15.VI, R6.2, TP8.PP
- new net N$37: IC15.ADJ, R20.1, R21.2
- new net N$39: C14.+, IC12.REF, IC12.VDD, IC13.OUT, TP10.PP
- new net N$40: IC12.SCLK, SV1.11
- new net N$41: IC11.OUT, R22.2, TP12.PP, X2.1
- new net N$42: IC12.SDATA, SV1.13
- new net N$44: IC11.IN-, R22.1, R23.2
- new net N$45: IC12.!CS, SV1.9
- new net N$47: IC11.IN+, IC12.FB, IC12.VOUT, TP11.PP
- new net N$51: B2.AC2, J2-1.S
- new net N$7: R26.1, SV1.4
- net GND: now also B2.-, C10.2, C11.-, C12.2, C13.-, C14.-, C9.-, IC11.-VS, IC12.GND, IC13.GND, R21.1, R23.1, R7.1, SV1.17, SV1.18, X2.2
- net N$8: now also SV1.7
Other:
- moved on the sheet: B2, C10, C11, C12, C13, C18, C9, IC11, IC12, IC13, IC14, IC15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

Commit message: compleat? version 0.1 first
Parts:
- added JP1: (no value), afc-smm:PINHD-1X1
- added S1: (no value), switch-omron:10-XX
- R24, R25: device rcl:R-TRIMM3296W -> afc-smm:R-TRIMM3296W
- SV1: device con-lstb:MA10-2W -> afc-smm:MA10-2W
Connections:
- new net N$55: S1.S, S1.S1, SV1.6
- net GND: now also JP1.1, R24.A, S1.P, S1.P1; no longer R25.A
- net N$13: now also R25.A, R25.S; no longer R24.A, R24.S
- net N$17: now also R24.S; no longer R25.S
- net N$18: now also R24.E; no longer R25.E
- net N$9: now also R25.E; no longer R24.E
Other:
- moved on the sheet: R24, R25

Commit message: add component value
Parts:
- C1, C11, C13, C2, C3, C4, C5, C9: value (none) -> 100u
- C10, C12, C16, C17, C6, C7, C8: value (none) -> 0.1
- C14, C18: value (none) -> 10u
- C19: value (none) -> 1.0u
- R1: value (none) -> 499
- R10: value (none) -> 1M
- R11: value (none) -> 750k
- R12, R13, R16, R23: value (none) -> 10k
- R14: value (none) -> 7k5
- R15: value (none) -> 3k
- R17, R24, R25, R8, R9: value (none) -> 100k
- R18: value (none) -> 2k
- R19: value (none) -> 10
- R2, R20, R5, R6: value (none) -> 240
- R21: value (none) -> 750
- R22: value (none) -> 75k
- R26, R27: value (none) -> 1k
- R3, R4: value (none) -> 2k2
- R7: value (none) -> 5k6
- X1, X2: value 1-227161-0 -> BNC-206
Connections:
- net +5V: now also C8.1; no longer C8.2
- net GND: now also C8.2; no longer C8.1
Other:
- moved on the sheet: C8, C9, R13, R17, R25, TP6

Commit message: it is work! go to add pid_controller
Connections:
- net N$34 renamed 30V
Other:
- moved on the sheet: B1, B2, C1, C10, C11, C12, C13, C14, C16, C17, C18, C19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
